Commit message: sensors load but not publish

File: dev_ws/install/solara_pkg/share/solara_pkg/description/gazebo.xacro (robot description, xacro)
@@ -61,120 +61,4 @@
         </visual>
     </gazebo>
-    <!-- IMU Sensor Gazebo Configuration -->
-    <gazebo reference="imu_link">
-        <sensor name="imu_sensor" type="imu">
-            <always_on>true</always_on>
-            <update_rate>100</update_rate>
-            <imu>
-                <angular_velocity>
-                    <x>
-                        <noise type="gaussian">
-                            <mean>0.0</mean>
-                            <stddev>0.0002</stddev>
-                        </noise>
-                    </x>
-                    <y>
-                        <noise type="gaussian">
-                            <mean>0.0</mean>
-                            <stddev>0.0002</stddev>
-                        </noise>
-                    </y>
-                    <z>
-                        <noise type="gaussian">
-                            <mean>0.0</mean>
-                            <stddev>0.0002</stddev>
-                        </noise>
-                    </z>
-                </angular_velocity>
-                <linear_acceleration>
-                    <x>
-                        <noise type="gaussian">
-                            <mean>0.0</mean>
-                            <stddev>0.017</stddev>
-                        </noise>
-                    </x>
-                    <y>
-                        <noise type="gaussian">
-                            <mean>0.0</mean>
-                            <stddev>0.017</stddev>
-                        </noise>
-                    </y>
-                    <z>
-                        <noise type="gaussian">
-                            <mean>0.0</mean>
-                            <stddev>0.017</stddev>
-                        </noise>
-                    </z>
-                </linear_acceleration>
-            </imu>
-        </sensor>
-    </gazebo>
-    <gazebo reference="ultrasonic_link">
-        <sensor name="ultrasonic" type="ray">
-        <always_on>true</always_on>
-        <update_rate>40</update_rate>
-        <visualize>true</visualize>
-        <topic>ultrasonic</topic>
-        <ray>
-            <scan>
-                <horizontal>
-                    <samples>5</samples>
-                    <resolution>1</resolution>
-                    <min_angle>-0.13</min_angle>  <!-- ~15° beam width -->
-                    <max_angle>0.13</max_angle>
-                </horizontal>
-            </scan>
-            <range>
-                <min>0.02</min>   <!-- 2cm minimum (HC-SR04 spec) -->
-                <max>4.0</max>    <!-- 4m maximum (HC-SR04 spec) -->
-                <resolution>0.01</resolution>  <!-- 1cm resolution -->
-            </range>
-            <noise>
-                <type>gaussian</type>
-                <mean>0.0</mean>
-                <stddev>0.01</stddev>  <!-- 1cm standard deviation -->
-            </noise>
-        </ray>
-        </sensor>
-    </gazebo>
-    <gazebo reference="gps_link">
-        <sensor name="gps_sensor" type="navsat">
-            <always_on>true</always_on>
-            <update_rate>10</update_rate>
-            <topic>gps</topic>
-            <navsat>
-                <position_sensing>
-                    <horizontal>
-                        <!-- 0.5m accuracy (better than standard NEO-M8N) -->
-                        <noise type="gaussian">
-                            <mean>0.0</mean>
-                            <stddev>0.5</stddev>
-                        </noise>
-                    </horizontal>
-                    <vertical>
-                        <!-- 1.5m vertical (still worse than horizontal) -->
-                        <noise type="gaussian">
-                            <mean>0.0</mean>
-                            <stddev>1.5</stddev>
-                        </noise>
-                    </vertical>
-                </position_sensing>
-                <velocity_sensing>
-                    <horizontal>
-                        <noise type="gaussian">
-                            <mean>0.0</mean>
-                            <stddev>0.1</stddev>
-                        </noise>
-                    </horizontal>
-                    <vertical>
-                        <noise type="gaussian">
-                            <mean>0.0</mean>
-                            <stddev>0.15</stddev>
-                        </noise>
-                    </vertical>
-                </velocity_sensing>
-            </navsat>
-        </sensor>
-    </gazebo>
     <!-- Gazebo Harmonic Diff Drive Plugin -->
     <gazebo>
@@ -191,3 +75,78 @@
         </plugin>
     </gazebo>
+    <!-- IMU Sensor -->
+<gazebo reference="imu_link">
+    <sensor name="imu_sensor" type="imu">
+        <always_on>true</always_on>
+        <update_rate>100</update_rate>
+        <topic>imu</topic>
+        <imu>
+            <angular_velocity>
+                <x><noise type="gaussian"><mean>0.0</mean><stddev>0.0002</stddev></noise></x>
+                <y><noise type="gaussian"><mean>0.0</mean><stddev>0.0002</stddev></noise></y>
+                <z><noise type="gaussian"><mean>0.0</mean><stddev>0.0002</stddev></noise></z>
+            </angular_velocity>
+            <linear_acceleration>
+                <x><noise type="gaussian"><mean>0.0</mean><stddev>0.017</stddev></noise></x>
+                <y><noise type="gaussian"><mean>0.0</mean><stddev>0.017</stddev></noise></y>
+                <z><noise type="gaussian"><mean>0.0</mean><stddev>0.017</stddev></noise></z>
+            </linear_acceleration>
+        </imu>
+    </sensor>
+</gazebo>
+<!-- Ultrasonic Sensor -->
+<gazebo reference="ultrasonic_link">
+    <sensor name="ultrasonic" type="ray">
+        <always_on>true</always_on>
+        <update_rate>40</update_rate>
+        <visualize>true</visualize>
+        <topic>ultrasonic</topic>
+        <ray>
+            <scan>
+                <horizontal>
+                    <samples>5</samples>
+                    <resolution>1</resolution>
+                    <min_angle>-0.13</min_angle>
+                    <max_angle>0.13</max_angle>
+                </horizontal>
+            </scan>
+            <range>
+                <min>0.02</min>
+                <max>4.0</max>
+                <resolution>0.01</resolution>
+            </range>
+            <noise>
+                <type>gaussian</type>
+                <mean>0.0</mean>
+                <stddev>0.01</stddev>
+            </noise>
+        </ray>
+    </sensor>
+</gazebo>
+<!-- GPS Sensor -->
+<gazebo reference="gps_link">
+    <sensor name="gps_sensor" type="navsat">
+        <always_on>true</always_on>
+        <update_rate>10</update_rate>
+        <topic>gps/fix</topic>
+        <navsat>
+            <position_sensing>
+                <horizontal>
+                    <noise type="gaussian"><mean>0.0</mean><stddev>0.5</stddev></noise>
+                </horizontal>
+                <vertical>
+                    <noise type="gaussian"><mean>0.0</mean><stddev>1.5</stddev></noise>
+                </vertical>
+            </position_sensing>
+            <velocity_sensing>
+                <horizontal>
+                    <noise type="gaussian"><mean>0.0</mean><stddev>0.1</stddev></noise>
+                </horizontal>
+                <vertical>
+                    <noise type="gaussian"><mean>0.0</mean><stddev>0.15</stddev></noise>
+                </vertical>
+            </velocity_sensing>
+        </navsat>
+    </sensor>
+</gazebo>
 </robot>

File: dev_ws/install/solara_pkg/share/solara_pkg/description/robot.urdf.xacro (robot description, xacro)
@@ -6,8 +6,8 @@
   <xacro:include filename="$(find solara_pkg)/description/chassis.xacro"/>
   <xacro:include filename="$(find solara_pkg)/description/wheels.xacro"/>
-  <xacro:include filename="$(find solara_pkg)/description/gazebo.xacro"/>
   <xacro:include filename="$(find solara_pkg)/description/sensors/imu.xacro"/>
   <xacro:include filename="$(find solara_pkg)/description/sensors/ultrasonic.xacro"/>
   <xacro:include filename="$(find solara_pkg)/description/sensors/gps.xacro"/>
+  <xacro:include filename="$(find solara_pkg)/description/gazebo.xacro"/>
   <!-- Assemble the robot: 2 driven + 4 passive wheels -->
   <xacro:driven_wheel prefix="middle_left" reflect_y="1"/>

File: dev_ws/install/solara_pkg/share/solara_pkg/description/sensors/gps.xacro (robot description, xacro)
@@ -22,9 +22,9 @@
     </collision>
     <inertial>
-        <mass value="0.010"/>
+        <mass value="0.5"/>
         <origin xyz="0 0 0" rpy="0 0 0"/>
-        <inertia ixx="0.000001" ixy="0.0" ixz="0.0"
-                 iyy="0.000001" iyz="0.0"
-                 izz="0.000001"/>
+        <inertia ixx="0.0001" ixy="0.0" ixz="0.0"
+                iyy="0.0001" iyz="0.0"
+                izz="0.0001"/>
     </inertial>
 </link>

File: dev_ws/install/solara_pkg/share/solara_pkg/description/sensors/imu.xacro (robot description, xacro)
@@ -18,10 +18,10 @@
                 </geometry>
             </collision>
-            <inertial>
-                <mass value="0.015"/>
+           <inertial>
+                <mass value="0.5"/>
                 <origin xyz="0 0 0" rpy="0 0 0"/>
-                <inertia ixx="0.00001" ixy="0.0" ixz="0.0"
-                         iyy="0.00001" iyz="0.0"
-                         izz="0.00001"/>
+                <inertia ixx="0.0001" ixy="0.0" ixz="0.0"
+                        iyy="0.0001" iyz="0.0"
+                        izz="0.0001"/>
             </inertial>
         </link>

File: dev_ws/install/solara_pkg/share/solara_pkg/description/sensors/ultrasonic.xacro (robot description, xacro)
@@ -20,9 +20,9 @@
         </collision>
         <inertial>
-            <mass value="0.003"/>  <!-- 3 grams -->
+            <mass value="0.5"/>
             <origin xyz="0 0 0" rpy="0 0 0"/>
-            <inertia ixx="0.000001" ixy="0.0" ixz="0.0"
-                    iyy="0.000001" iyz="0.0"
-                    izz="0.000001"/>
+            <inertia ixx="0.0001" ixy="0.0" ixz="0.0"
+                    iyy="0.0001" iyz="0.0"
+                    izz="0.0001"/>
         </inertial>
     </link>

Commit message: lidar

File: dev_ws/install/solara_pkg/share/solara_pkg/description/gazebo.xacro (robot description, xacro)
@@ -156,3 +156,33 @@
     </sensor>
 </gazebo>
+<gazebo reference="lidar_link">
+    <sensor name="gpu_lidar" type="gpu_lidar">
+        <always_on>true</always_on>
+        <update_rate>10</update_rate>
+        <topic>scan</topic>
+        <gz_frame_id>lidar_link</gz_frame_id>
+        <ray>
+            <scan>
+                <horizontal>
+                    <samples>360</samples>
+                    <resolution>1</resolution>
+                    <min_angle>-3.14159</min_angle>
+                    <max_angle>3.14159</max_angle>
+                </horizontal>
+                <vertical>
+                    <samples>1</samples>
+                    <resolution>1</resolution>
+                    <min_angle>0</min_angle>
+                    <max_angle>0</max_angle>
+                </vertical>
+            </scan>
+            <range>
+                <min>0.15</min>
+                <max>12.0</max>
+                <resolution>0.01</resolution>
+            </range>
+        </ray>
+        <visualize>true</visualize>
+    </sensor>
+</gazebo>
 </robot>

File: dev_ws/install/solara_pkg/share/solara_pkg/description/robot.urdf.xacro (robot description, xacro)
@@ -8,4 +8,5 @@
   <xacro:include filename="$(find solara_pkg)/description/sensors/imu.xacro"/>
   <xacro:include filename="$(find solara_pkg)/description/sensors/ultrasonic.xacro"/>
+  <xacro:include filename="$(find solara_pkg)/description/sensors/lidar.xacro"/>
   <xacro:include filename="$(find solara_pkg)/description/sensors/gps.xacro"/>
   <xacro:include filename="$(find solara_pkg)/description/gazebo.xacro"/>
@@ -27,4 +28,7 @@
     <origin xyz="0.2 0.1 0.0862" rpy="0 0 0"/>
   </xacro:gps_sensor>
+  <xacro:lidar_sensor parent_link="base_link">
+    <origin xyz="0.2 0 0.1" rpy="0 0 0"/>
+  </xacro:lidar_sensor>
   <!-- add your lidar tag here -->
 </robot>
