Commit message: test nav2

File: install/solara_pkg/share/solara_pkg/description/gazebo.xacro (robot description, xacro)
@@ -75,56 +75,33 @@
         </plugin>
     </gazebo>
-      <!-- IMU Sensor Gazebo Configuration -->
-    <gazebo reference="base_link">
-        <sensor name="imu_sensor" type="imu">
-            <always_on>true</always_on>
-            <update_rate>100</update_rate>
-            <topic>imu</topic>
-            <imu>
-                <angular_velocity>
-                    <x>
-                        <noise type="gaussian">
-                            <mean>0.0</mean>
-                            <stddev>0.0002</stddev>
-                        </noise>
-                    </x>
-                    <y>
-                        <noise type="gaussian">
-                            <mean>0.0</mean>
-                            <stddev>0.0002</stddev>
-                        </noise>
-                    </y>
-                    <z>
-                        <noise type="gaussian">
-                            <mean>0.0</mean>
-                            <stddev>0.0002</stddev>
-                        </noise>
-                    </z>
-                </angular_velocity>
-                <linear_acceleration>
-                    <x>
-                        <noise type="gaussian">
-                            <mean>0.0</mean>
-                            <stddev>0.017</stddev>
-                        </noise>
-                    </x>
-                    <y>
-                        <noise type="gaussian">
-                            <mean>0.0</mean>
-                            <stddev>0.017</stddev>
-                        </noise>
-                    </y>
-                    <z>
-                        <noise type="gaussian">
-                            <mean>0.0</mean>
-                            <stddev>0.017</stddev>
-                        </noise>
-                    </z>
-                </linear_acceleration>
-            </imu>
-        </sensor>
+    <!-- Joint State Publisher -->
+    <gazebo>
+        <plugin filename="gz-sim-joint-state-publisher-system"
+                name="gz::sim::systems::JointStatePublisher">
+        </plugin>
     </gazebo>
-    <gazebo reference="base_link">
-        <sensor name="ultrasonic" type="ray">
+    <!-- IMU Sensor -->
+<gazebo reference="imu_link">
+    <sensor name="imu_sensor" type="imu">
+        <always_on>true</always_on>
+        <update_rate>100</update_rate>
+        <topic>imu</topic>
+        <imu>
+            <angular_velocity>
+                <x><noise type="gaussian"><mean>0.0</mean><stddev>0.0002</stddev></noise></x>
+                <y><noise type="gaussian"><mean>0.0</mean><stddev>0.0002</stddev></noise></y>
+                <z><noise type="gaussian"><mean>0.0</mean><stddev>0.0002</stddev></noise></z>
+            </angular_velocity>
+            <linear_acceleration>
+                <x><noise type="gaussian"><mean>0.0</mean><stddev>0.017</stddev></noise></x>
+                <y><noise type="gaussian"><mean>0.0</mean><stddev>0.017</stddev></noise></y>
+                <z><noise type="gaussian"><mean>0.0</mean><stddev>0.017</stddev></noise></z>
+            </linear_acceleration>
+        </imu>
+    </sensor>
+</gazebo>
+<!-- Ultrasonic Sensor -->
+<gazebo reference="ultrasonic_link">
+    <sensor name="ultrasonic" type="ray">
         <always_on>true</always_on>
         <update_rate>40</update_rate>
@@ -136,59 +113,76 @@
                     <samples>5</samples>
                     <resolution>1</resolution>
-                    <min_angle>-0.13</min_angle>  <!-- ~15° beam width -->
+                    <min_angle>-0.13</min_angle>
                     <max_angle>0.13</max_angle>
                 </horizontal>
             </scan>
             <range>
-                <min>0.02</min>   <!-- 2cm minimum (HC-SR04 spec) -->
-                <max>4.0</max>    <!-- 4m maximum (HC-SR04 spec) -->
-                <resolution>0.01</resolution>  <!-- 1cm resolution -->
+                <min>0.02</min>
+                <max>4.0</max>
+                <resolution>0.01</resolution>
             </range>
             <noise>
                 <type>gaussian</type>
                 <mean>0.0</mean>
-                <stddev>0.01</stddev>  <!-- 1cm standard deviation -->
+                <stddev>0.01</stddev>
             </noise>
         </ray>
-        </sensor>
-    </gazebo>
-    <gazebo reference="base_link">
-        <sensor name="gps_sensor" type="navsat">
-            <always_on>true</always_on>
-            <update_rate>10</update_rate>
-            <topic>gps/fix</topic>
-            <navsat>
-                <position_sensing>
-                    <horizontal>
-                        <!-- 0.5m accuracy (better than standard NEO-M8N) -->
-                        <noise type="gaussian">
-                            <mean>0.0</mean>
-                            <stddev>0.5</stddev>
-                        </noise>
-                    </horizontal>
-                    <vertical>
-                        <!-- 1.5m vertical (still worse than horizontal) -->
-                        <noise type="gaussian">
-                            <mean>0.0</mean>
-                            <stddev>1.5</stddev>
-                        </noise>
-                    </vertical>
-                </position_sensing>
-                <velocity_sensing>
-                    <horizontal>
-                        <noise type="gaussian">
-                            <mean>0.0</mean>
-                            <stddev>0.1</stddev>
-                        </noise>
-                    </horizontal>
-                    <vertical>
-                        <noise type="gaussian">
-                            <mean>0.0</mean>
-                            <stddev>0.15</stddev>
-                        </noise>
-                    </vertical>
-                </velocity_sensing>
-            </navsat>
-        </sensor>
-    </gazebo>
+    </sensor>
+</gazebo>
+<!-- GPS Sensor -->
+<gazebo reference="gps_link">
+    <sensor name="gps_sensor" type="navsat">
+        <always_on>true</always_on>
+        <update_rate>10</update_rate>
+        <topic>gps/fix</topic>
+        <navsat>
+            <position_sensing>
+                <horizontal>
+                    <noise type="gaussian"><mean>0.0</mean><stddev>0.5</stddev></noise>
+                </horizontal>
+                <vertical>
+                    <noise type="gaussian"><mean>0.0</mean><stddev>1.5</stddev></noise>
+                </vertical>
+            </position_sensing>
+            <velocity_sensing>
+                <horizontal>
+                    <noise type="gaussian"><mean>0.0</mean><stddev>0.1</stddev></noise>
+                </horizontal>
+                <vertical>
+                    <noise type="gaussian"><mean>0.0</mean><stddev>0.15</stddev></noise>
+                </vertical>
+            </velocity_sensing>
+        </navsat>
+    </sensor>
+</gazebo>
+<gazebo reference="lidar_link">
+    <sensor name="gpu_lidar" type="gpu_lidar">
+        <always_on>true</always_on>
+        <update_rate>10</update_rate>
+        <topic>scan</topic>
+        <gz_frame_id>lidar_link</gz_frame_id>
+        <ray>
+            <scan>
+                <horizontal>
+                    <samples>360</samples>
+                    <resolution>1</resolution>
+                    <min_angle>-3.14159</min_angle>
+                    <max_angle>3.14159</max_angle>
+                </horizontal>
+                <vertical>
+                    <samples>1</samples>
+                    <resolution>1</resolution>
+                    <min_angle>0</min_angle>
+                    <max_angle>0</max_angle>
+                </vertical>
+            </scan>
+            <range>
+                <min>0.15</min>
+                <max>12.0</max>
+                <resolution>0.01</resolution>
+            </range>
+        </ray>
+        <visualize>true</visualize>
+    </sensor>
+</gazebo>
 </robot>

File: install/solara_pkg/share/solara_pkg/description/robot.urdf.xacro (robot description, xacro)
@@ -8,4 +8,5 @@
   <xacro:include filename="$(find solara_pkg)/description/sensors/imu.xacro"/>
   <xacro:include filename="$(find solara_pkg)/description/sensors/ultrasonic.xacro"/>
+  <xacro:include filename="$(find solara_pkg)/description/sensors/lidar.xacro"/>
   <xacro:include filename="$(find solara_pkg)/description/sensors/gps.xacro"/>
   <xacro:include filename="$(find solara_pkg)/description/gazebo.xacro"/>
@@ -27,4 +28,7 @@
     <origin xyz="0.2 0.1 0.0862" rpy="0 0 0"/>
   </xacro:gps_sensor>
+  <xacro:lidar_sensor parent_link="base_link">
+    <origin xyz="0.2 0 0.1" rpy="0 0 0"/>
+  </xacro:lidar_sensor>
   <!-- add your lidar tag here -->
 </robot>
